File: EL6050_project/pcb.sch (EAGLE design)
At the start: 6 parts

Commit message: add lorawan module and arduino to schematic
Parts:
- added H1, H2, H3, H4: MOUNT-HOLE3.2, holes:MOUNT-HOLE3.2
- added IC1: MEGA8-P, atmel:MEGA8-P
- added R1, R2, R3, R4, R5, R6: (no value), rcl:R-EU_R1206W
- added U$1: MICROCHIP_RN2483, lora-lorawan-modules:MICROCHIP_RN2483
Connections:
- new net N$1: U$1.GPIO0
- new net N$10: U$1.GPIO4
- new net N$11: U$1.GPIO6
- new net N$12: U$1.GPIO8
- new net N$13: U$1.GPIO9
- new net N$14: U$1.GPIO12
- new net N$15: U$1.VDD
- new net N$16: U$1.RESET
- new net N$17: U$1.RFL
- new net N$18: U$1.UART_CTS
- new net N$19: U$1.UART_RX
- new net N$2: U$1.GPIO1
- new net N$20: U$1.PGD_INT
- new net N$21: U$1.GND
- new net N$22: U$1.RFH
- new net N$23: U$1.UART_RTS
- new net N$24: U$1.UART_TX
- new net N$25: U$1.PGC_INT
- new net N$26: LED1.C
- new net N$27: LED2.C
- new net N$28: LED3.C
- new net N$29: LED4.C
- new net N$3: U$1.GPIO2
- new net N$30: LED5.C
- new net N$31: LED6.C
- new net N$32: LED1.A, R1.1
- new net N$33: LED2.A, R2.1
- new net N$34: LED3.A, R3.1
- new net N$35: LED4.A, R4.1
- new net N$36: LED5.A, R5.1
- new net N$37: LED6.A, R6.1
- new net N$38: IC1.PC0(ADC0)
- new net N$39: IC1.PC2(ADC2)
- new net N$4: U$1.GPIO3
- new net N$40: IC1.PD0(RXD)
- new net N$41: IC1.PD2(INT0)
- new net N$42: IC1.PD4(XCK/T0)
- new net N$43: IC1.PD6(AIN0)
- new net N$44: IC1.PB0(ICP)
- new net N$45: IC1.PB3(MOSI/OC2)
- new net N$46: IC1.PB4(MISO)
- new net N$47: IC1.PC4(ADC4/SDA)
- new net N$48: IC1.PC1(ADC1)
- new net N$49: IC1.PC3(ADC3)
- new net N$5: U$1.GPIO5
- new net N$50: IC1.PC5(ADC5/SCL)
- new net N$51: IC1.PD1(TXD)
- new net N$52: IC1.PD3(INT1)
- new net N$53: IC1.PD5(T1)
- new net N$54: IC1.PD7(AIN1)
- new net N$55: IC1.PB1(OC1A)
- new net N$56: IC1.PB2(SS/OC1B)
- new net N$57: IC1.PB5(SCK)
- new net N$6: U$1.GPIO7
- new net N$7: U$1.GPIO10
- new net N$8: U$1.GPIO11
- new net N$9: U$1.GPIO13

Commit message: add and connect components
Parts:
- added C1, C2, C3, C4, C5, C6: (no value), rcl:C-EU050-025X075
- added IC2: MEGA8-P, atmel:MEGA8-P
- added Q1, Q2: (no value), crystal:CRYSTALHC18U-V
- added R10, R11, R7, R8: (no value), rcl:R-EU_R1206W
- added R9: 10k, rcl:R-EU_R1206W
- added SV1, SV2: (no value), con-lstb:MA03-1
- added X1: BU-SMA-V, con-coax:BU-SMA-V
- added X2: GMSTBA2, con-phoenix-762:GMSTBA2
Connections:
- new net 5V: C3.2, C6.2, IC1.VCC@1, IC2.VCC@1, R11.2, R8.2, SV1.1, SV2.1
- new net GND: C1.1, C2.1, C3.1, C4.1, C5.1, C6.1, IC1.GND@1, IC2.GND@1, LED4.A, R1.2, R2.2, R3.2, R4.1, R4.2, R5.2, R6.2, SV1.2, SV2.2, U$1.GND, X1.2
- new net N$58: IC1.PC6(/RESET), R8.1
- new net N$59: IC1.AREF
- new net N$60: C2.2, IC1.PB6(XTAL1/TOSC1), Q1.2, R7.2
- new net N$61: IC2.PB3(MOSI/OC2)
- new net N$62: IC1.GND
- new net N$63: IC1.AVCC
- new net N$64: C1.2, IC1.PB7(XTAL2/TOSC2), Q1.1, R7.1
- new net N$65: IC2.PB4(MISO)
- new net N$66: IC2.PC4(ADC4/SDA)
- new net N$67: IC2.PC1(ADC1)
- new net N$68: IC2.PC3(ADC3)
- new net N$69: IC2.PC5(ADC5/SCL)
- new net N$70: IC2.PD3(INT1)
- new net N$71: IC2.PD5(T1)
- new net N$72: IC2.PD7(AIN1)
- new net N$73: IC2.PB1(OC1A)
- new net N$74: IC2.PB2(SS/OC1B)
- new net N$75: IC2.PB5(SCK)
- new net N$76: IC2.PC6(/RESET), R11.1
- new net N$77: IC2.AREF
- new net N$78: C5.2, IC2.PB6(XTAL1/TOSC1), Q2.2, R10.2
- new net N$79: IC2.GND
- new net N$80: IC2.AVCC
- new net N$81: C4.2, IC2.PB7(XTAL2/TOSC2), Q2.1, R10.1
- new net RF_LRW: U$1.RFH, X1.1
- new net RX-LRW: IC1.PD0(RXD), IC2.PD0(RXD), U$1.UART_TX
- new net TX-LRW: IC1.PD1(TXD), IC2.PD1(TXD), U$1.UART_RX
- new net ULS1: SV1.3
- new net ULS2: SV2.3
- new net VCC: R9.1, U$1.VDD
- net N$15: now also X2-1.1; no longer U$1.VDD
- net N$16: now also R9.2
- net N$19: now also X2-2.1; no longer U$1.UART_RX
- net N$21: now also IC2.PC0(ADC0); no longer U$1.GND
- net N$22: now also IC2.PC2(ADC2); no longer U$1.RFH
- net N$24: now also IC2.PD2(INT0); no longer U$1.UART_TX
- net N$35: now also IC2.PD4(XCK/T0); no longer LED4.A, R4.1
- net N$40: now also IC2.PD6(AIN0); no longer IC1.PD0(RXD)
- net N$51: now also IC2.PB0(ICP); no longer IC1.PD1(TXD)

Commit message: all components added and board started
Parts:
- removed Q2: (no value), crystal:CRYSTALHC18U-V
- removed R10, R11: (no value), rcl:R-EU_R1206W
- removed SV1, SV2: (no value), con-lstb:MA03-1
- removed X1: BU-SMA-V, con-coax:BU-SMA-V
- removed X2: GMSTBA2, con-phoenix-762:GMSTBA2
- added ANTENA: BU-SMA-V, con-coax:BU-SMA-V
- added C10: 100n, rcl:C-EU050-024X044
- added C7: 100nF, rcl:C-EU050-025X075
- added C8: 0.1u, rcl:C-EU050-025X075
- added C9: 47u, rcl:CPOL-EUE2,5-6E
- added D1: 1N4004, diode:1N4004
- added FTDI: (no value), con-lstb:MA06-1
- added L1: 100mF, inductor-coilcraft2:MSS1260
- added LIDAR1, LIDAR2: (no value), sparkfun-connectors:CONN_04JST-PTH
- added POWERSUPPLY: (no value), con-phoenix-500:MSTBV2
- C3, C4, C5, C6: value (none) -> 100nF
- IC1: value MEGA8-P -> ATMEGA2560-16AU; device atmel:MEGA8-P -> atmel-2005:ATMEGA2560-16AU
- IC2: value MEGA8-P -> 7805T; device atmel:MEGA8-P -> linear:7805T
- R7: value (none) -> 1M
- R8: value (none) -> 10k
- renumbered U$1 to LRW-RN2903
Connections:
- net N$16 renamed RST-LRW
- removed net N$15: X2-1.1
- removed net N$19: X2-2.1
- removed net N$24: IC2.PD2(INT0)
- removed net N$26: LED1.C
- removed net N$27: LED2.C
- removed net N$28: LED3.C
- removed net N$29: LED4.C
- removed net N$30: LED5.C
- removed net N$31: LED6.C
- removed net N$35: IC2.PD4(XCK/T0)
- removed net N$38: IC1.PC0(ADC0)
- removed net N$39: IC1.PC2(ADC2)
- removed net N$40: IC2.PD6(AIN0)
- removed net N$43: IC1.PD6(AIN0)
- removed net N$44: IC1.PB0(ICP)
- removed net N$45: IC1.PB3(MOSI/OC2)
- removed net N$51: IC2.PB0(ICP)
- removed net N$55: IC1.PB1(OC1A)
- removed net N$59: IC1.AREF
- removed net N$61: IC2.PB3(MOSI/OC2)
- removed net N$65: IC2.PB4(MISO)
- removed net N$67: IC2.PC1(ADC1)
- removed net N$68: IC2.PC3(ADC3)
- removed net N$70: IC2.PD3(INT1)
- removed net N$71: IC2.PD5(T1)
- removed net N$72: IC2.PD7(AIN1)
- removed net N$73: IC2.PB1(OC1A)
- removed net N$74: IC2.PB2(SS/OC1B)
- removed net N$75: IC2.PB5(SCK)
- removed net N$76: IC2.PC6(/RESET), R11.1
- removed net N$77: IC2.AREF
- removed net N$78: C5.2, IC2.PB6(XTAL1/TOSC1), Q2.2, R10.2
- removed net N$79: IC2.GND
- removed net RF_LRW: LRW-RN2903.RFH, X1.1
- removed net ULS1: SV1.3
- removed net ULS2: SV2.3
- removed net VCC: LRW-RN2903.VDD, R9.1
- new net 3V3: FTDI.1, IC2.VO, LRW-RN2903.VDD, R9.1
- new net AVCC: C7.2, IC1.AVCC, L1.1
- new net DST-CP: C8.1, FTDI.6
- new net L_DIST: IC1.PL5(OC5C), LED6.C
- new net L_ON: IC1.PL7
- new net L_RED: IC1.PL6, LED2.C
- new net L_TRSA: IC1.PL4(OC5B), LED3.C
- new net L_TRSB: IC1.PL3(OC5A), LED4.C
- new net L_TRSC: IC1.PL2(T5), LED5.C
- new net N$100: IC1.(AD2)PA2
- new net N$101: IC1.(AD0)PA0
- new net N$102: IC1.(OC1B/PCINT6)PB6
- new net N$103: IC1.(OC2A/PCINT4)PB4
- new net N$104: IC1.(MOSI/PCINT2)PB2
- new net N$105: IC1.(SCK/PCINT1)PB1
- new net N$106: IC1.(A14)PC6
- new net N$107: IC1.(A12)PC4
- new net N$108: IC1.(A9)PC1
- new net N$109: IC1.(A8)PC0
- new net N$110: IC1.(T1)PD6
- new net N$111: IC1.(ICP1)PD4
- new net N$113: IC1.(SCL/INT0)PD0
- new net N$114: IC1.(T3/INT6)PE6
- new net N$115: IC1.(OC3B/INT4)PE4
- new net N$116: IC1.(XCK0/AIN0)PE2
- new net N$118: IC1.(ADC6/TDO)PF6
- new net N$119: IC1.(ADC4/TCK)PF4
- new net N$120: IC1.(ADC2)PF2
- new net N$121: IC1.(ADC0)PF0
- new net N$122: IC1.(TOSC1)PG4
- new net N$123: IC1.(ALE)PG2
- new net N$124: IC1.(WR)PG0
- new net N$125: IC1.(A10)PC2
- new net N$126: IC1.(T0)PD7
- new net N$127: IC1.(XCK1)PD5
- new net N$129: IC1.(SDA/INT1)PD1
- new net N$130: IC1.(CLKO/ICP3/INT7)PE7
- new net N$131: IC1.(OC3C/INT5)PE5
- new net N$132: IC1.(OC3A/AIN1)PE3
- new net N$134: IC1.(ADC7/TDI)PF7
- new net N$135: IC1.(ADC5/TMS)PF5
- new net N$136: IC1.(ADC3)PF3
- new net N$137: IC1.(ADC1)PF1
- new net N$138: IC1.(OC0B)PG5
- new net N$139: IC1.(TOSC2)PG3
- new net N$140: IC1.(RD)PG1
- new net N$82: IC1.(MISO/PCINT3)PB3
- new net N$83: IC1.(SS/PCINT0)PB0
- new net N$84: IC1.(A15)PC7
- new net N$85: IC1.(A13)PC5
- new net N$86: IC1.(A11)PC3
- new net N$87: IC1.PK4(ADC12/PCINT20)
- new net N$88: IC1.PK2(ADC10/PCINT18)
- new net N$89: IC1.PK0(ADC8/PCINT16)
- new net N$90: IC1.PJ6(PCINT15)
- new net N$91: IC1.PJ4(PCINT13)
- new net N$92: IC1.PJ2(XCK3/PCINT11)
- new net N$94: IC1.PH6(OC2B)
- new net N$95: IC1.PH4(OC4B)
- new net N$96: IC1.PH2(XCK2)
- new net N$98: IC1.(AD6)PA6
- new net N$99: IC1.(AD4)PA4
- new net PWRIN: D1.A, POWERSUPPLY-1.SK
- new net RF-LRW: ANTENA.1, LRW-RN2903.RFH
- new net RX-CP: FTDI.5, IC1.PJ1(TXD3/PCINT10)
- new net RX-LID1: IC1.(TXD1/INT3)PD3, LIDAR1.2
- new net RX-LID2: IC1.PH1(TXD2), LIDAR2.2
- new net TX-CP: FTDI.4, IC1.PJ0(RXD3/PCINT9)
- new net TX-LID1: IC1.(RXD1/INT2)PD2, LIDAR1.1
- new net TX-LID2: IC1.PH0(RXD2), LIDAR2.1
- net 5V: now also C10.1, C4.2, C5.2, C9.+, D1.C, FTDI.3, IC1.VCC, IC1.VCC1, IC1.VCC2, IC1.VCC3, IC2.VI, L1.2, LED1.C, LIDAR1.3, LIDAR2.3, R8.1; no longer C6.2, IC1.VCC@1, IC2.VCC@1, R11.2, R8.2, SV1.1, SV2.1
- net GND: now also ANTENA.2, C10.2, C6.2, C7.1, C9.-, FTDI.2, IC1.AGND, IC1.GND, IC1.GND1, IC1.GND2, IC1.GND3, IC2.GND, LIDAR1.4, LIDAR2.4, POWERSUPPLY-2.SK; no longer C6.1, IC1.GND@1, IC2.GND@1, SV1.2, SV2.2, X1.2
- net N$21: now also C8.2, IC1.RESET, R8.2; no longer IC2.PC0(ADC0)
- net N$22: now also C6.1, IC1.AREF; no longer IC2.PC2(ADC2)
- net N$41: now also C1.2, IC1.XTAL1, Q1.1, R7.1; no longer IC1.PD2(INT0)
- net N$42: now also C2.2, IC1.XTAL2, Q1.2, R7.2; no longer IC1.PD4(XCK/T0)
- net N$46: now also IC1.PL1(ICP5); no longer IC1.PB4(MISO)
- net N$47: now also IC1.PK7(ADC15/PCINT23); no longer IC1.PC4(ADC4/SDA)
- net N$48: now also IC1.PK5(ADC13/PCINT21); no longer IC1.PC1(ADC1)
- net N$49: now also IC1.PK3(ADC11/PCINT19); no longer IC1.PC3(ADC3)
- net N$50: now also IC1.PK1(ADC9/PCINT17); no longer IC1.PC5(ADC5/SCL)
- net N$52: now also IC1.PJ7; no longer IC1.PD3(INT1)
- net N$53: now also IC1.PJ5(PCINT14); no longer IC1.PD5(T1)
- net N$54: now also IC1.PJ3(PCINT12); no longer IC1.PD7(AIN1)
- net N$56: now also IC1.PH7(T4); no longer IC1.PB2(SS/OC1B)
- net N$57: now also IC1.PH5(OC4C); no longer IC1.PB5(SCK)
- net N$58: now also IC1.PH3(OC4A); no longer IC1.PC6(/RESET), R8.1
- net N$60: now also IC1.(AD7)PA7; no longer C2.2, IC1.PB6(XTAL1/TOSC1), Q1.2, R7.2
- net N$62: now also IC1.(AD5)PA5; no longer IC1.GND
- net N$63: now also IC1.(AD3)PA3; no longer IC1.AVCC
- net N$64: now also IC1.(AD1)PA1; no longer C1.2, IC1.PB7(XTAL2/TOSC2), Q1.1, R7.1
- net N$66: now also IC1.(OC0A/OC1C/PCINT7)PB7; no longer IC2.PC4(ADC4/SDA)
- net N$69: now also IC1.(OC1A/PCINT5)PB5; no longer IC2.PC5(ADC5/SCL)
- net N$80: now also IC1.PL0(ICP4); no longer IC2.AVCC
- net N$81: now also IC1.PK6(ADC14/PCINT22); no longer C4.2, IC2.PB7(XTAL2/TOSC2), Q2.1, R10.1
- net RX-LRW: now also IC1.(TXD0)PE1, LRW-RN2903.UART_RX; no longer IC1.PD0(RXD), IC2.PD0(RXD), LRW-RN2903.UART_TX
- net TX-LRW: now also IC1.(RXD0/PCIN8)PE0, LRW-RN2903.UART_TX; no longer IC1.PD1(TXD), IC2.PD1(TXD), LRW-RN2903.UART_RX

Commit message: end board and update schematic
Parts:
- removed LED1, LED2, LED3, LED4, LED5, LED6: (no value), adafruit:LED5MM
- removed POWERSUPPLY: (no value), con-phoenix-500:MSTBV2
- added C11, C12: 10u, rcl:CPOL-EUE2,5-6E
- added D2, D3, D4, D5, D6, D7, D8, D9: 1N4004, diode:1N4004
- added IC3: 7805T, linear:7805T
- added J1: DCJ0202, con-jack:DCJ0202
- added L_5V, L_DIST, L_RED, L_TRSA, L_TRSB, L_TRSC: (no value), adafruit:LED5MM
- added R10, R11: 10k, rcl:R-EU_R1206W
- added TRSA, TRSB, TRSC: (no value), sparkfun-connectors:CONN_04JST-PTH
- added U1: LM358, sparkfun-amplifiers:LM358
- C1, C2: value (none) -> 22p
- C10: value 100n -> 47u; device rcl:C-EU050-024X044 -> rcl:CPOL-EUE2,5-6E
- C3, C4, C5, C6, C7: value 100nF -> 100n
- C8: value 0.1u -> 100n
- IC2: VOUT (none) -> 5V
- L1: value 100mF -> 10u
- Q1: value (none) -> 16MHz
- R1, R2, R3, R4, R5, R6: value (none) -> 100
Connections:
- net N$21 renamed RESET
- net N$41 renamed XTAL1
- net N$42 renamed XTAL2
- removed net N$108: IC1.(A9)PC1
- removed net N$109: IC1.(A8)PC0
- removed net N$125: IC1.(A10)PC2
- new net -15V: R11.2, TRSA.3, TRSB.3, TRSC.3, U1G1.OUT
- new net 15V: C10.+, D2.C, D3.C, IC2.VI, R10.1, TRSA.4, TRSB.4, TRSC.4, U1G3.P$V+
- new net N$15: R10.2, R11.1, U1G1.-IN
- new net N$16: L_TRSB.A, R4.1
- new net VO_A: D4.C, D5.A, IC1.(A10)PC2, TRSA.2
- new net VO_B: D6.C, D7.A, IC1.(A9)PC1, TRSB.2
- new net VO_C: D8.C, D9.A, IC1.(A8)PC0, TRSC.2
- net 3V3: now also C11.+, D1.A, IC3.VO; no longer IC2.VO
- net 5V: now also C12.+, D2.A, D5.C, D7.C, D9.C, IC2.VO, IC3.VI, L_5V.C; no longer C10.1, IC2.VI, LED1.C
- net GND: now also C10.-, C11.-, C12.-, D4.A, D6.A, D8.A, IC3.GND, J1.2, J1.3, TRSA.1, TRSB.1, TRSC.1, U1G1.+IN, U1G3.P$V-; no longer C10.2, LED4.A, POWERSUPPLY-2.SK, R4.1
- net L_DIST: now also L_DIST.C; no longer LED6.C
- net L_RED: now also L_RED.C; no longer LED2.C
- net L_TRSA: now also L_TRSA.C; no longer LED3.C
- net L_TRSB: now also L_TRSB.C; no longer LED4.C
- net L_TRSC: now also L_TRSC.C; no longer LED5.C
- net N$32: now also L_5V.A; no longer LED1.A
- net N$33: now also L_RED.A; no longer LED2.A
- net N$34: now also L_TRSA.A; no longer LED3.A
- net N$36: now also L_TRSC.A; no longer LED5.A
- net N$37: now also L_DIST.A; no longer LED6.A
- net PWRIN: now also D3.A, J1.1; no longer D1.A, POWERSUPPLY-1.SK
