File: T3/pcb.brd (EAGLE design)
At the start: 91.7 x 73.3 mm, 57 parts, among them IC1 ATMEGA2560-16AU, IC2 7805T, IC3 7805T, J1 DCJ0202, Q1 16MHz, U1 LM358

Commit message: hardware complete
Parts:
- added Q2, Q3: (no value), adafruit:SOT23-W
- added R12, R13, R14, R15: 10k, rcl_mod:R1206W
- R1, R10, R11, R2, R3, R4, R5, R6, R8: device rcl:R1206W -> rcl_mod:R1206W
- moved C6 27.0 mm to (41.9, 68.3), turned to 0 degrees
- moved C7 6.98 mm to (51.8, 41.3)
- moved C3 6.67 mm to (55.2, 41.3)
- moved C4 6.35 mm to (58.7, 41.3)
- moved C5 6.03 mm to (62.2, 41.3)
- moved C11 4.76 mm to (33.3, 6.99)
- moved C12 4.76 mm to (23.2, 6.99)
- moved D1 4.76 mm to (28.3, 12.4)
- moved IC3 4.76 mm to (28.3, 27.6)
- renumbered FTDI to USB-SERIAL
Connections:
- new net N$19: USB-SERIAL.1
- new net RX-LRW5V: IC1.3, Q2.3, R13.2
- new net TX-LRW5V: IC1.2, Q3.3, R15.2
- net 3V3: now also Q2.1, Q3.1, R12.1, R14.1; no longer USB-SERIAL.1
- net 5V: now also R13.1, R15.1; no longer L_5V.K
- net L_ON: now also L_5V.K
- net RX-LRW: now also Q2.2, R12.2; no longer IC1.3
- net TX-LRW: now also Q3.2, R14.2; no longer IC1.2
Routing:
- net GND: track 465.3 -> 296.1 mm, vias 1 -> 0
- net L_ON: track 0.00 -> 55.8 mm, vias 0 -> 1
- net 5V: track 309.9 -> 353.3 mm, vias 1 -> 5
- net RX-LRW5V: track 0.00 -> 34.6 mm
- net 3V3: track 122.8 -> 98.4 mm, vias 1 -> 2
- net N$22: track 8.35 -> 19.5 mm
- net TX-LRW5V: track 0.00 -> 10.6 mm
- net TX-LRW: track 9.91 -> 19.5 mm
- net AVCC: track 26.9 -> 35.2 mm, vias 2 -> 3
- net RX-LRW: track 9.98 -> 17.6 mm
- net 15V: track 146.5 -> 141.7 mm
- net RX-LID1: track 63.7 -> 64.8 mm
- net L_TRSA: track 71.0 -> 72.1 mm
- net RX-LID2: track 59.6 -> 60.4 mm
- net L_TRSB: track 65.8 -> 66.4 mm
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- added copper zone on layer 1, net GND
- added copper zone on layer 16, net GND
Other:
- board size 91.7 x 73.3 mm -> 91.7 x 73.6 mm
