File: T3/pcb.sch (EAGLE design)
At the start: 57 parts, among them IC1 ATMEGA2560-16AU, IC2 7805T, IC3 7805T, J1 DCJ0202, Q1 16MHz, U1 LM358

Commit message: hardware complete
Parts:
- added Q2, Q3: (no value), adafruit:MOSFET-NWAVE
- added R12, R13, R14, R15: 10k, rcl_mod:R-EU_R1206W
- R1, R10, R11, R2, R3, R4, R5, R6, R8: device rcl:R-EU_R1206W -> rcl_mod:R-EU_R1206W
- renumbered FTDI to USB-SERIAL
Connections:
- new net N$19: USB-SERIAL.1
- new net RX-LRW5V: IC1.(TXD0)PE1, Q2.D, R13.2
- new net TX-LRW5V: IC1.(RXD0/PCIN8)PE0, Q3.D, R15.2
- net 3V3: now also Q2.G, Q3.G, R12.1, R14.1; no longer USB-SERIAL.1
- net 5V: now also R13.1, R15.1; no longer L_5V.C
- net L_ON: now also L_5V.C
- net RX-LRW: now also Q2.S, R12.2; no longer IC1.(TXD0)PE1
- net TX-LRW: now also Q3.S, R14.2; no longer IC1.(RXD0/PCIN8)PE0
Other:
- moved on the sheet: ANTENA
